Commit message: sim ready to use with minor bugs

File: ros2_ws/src/webots_ros2_suv/resource/vesta.urdf (robot description, URDF)
Before this commit: robot vesta, 0 links, 0 joints
Links:
- added link base_link
- added link body_link; visual box size=1.41 1.73 0.78; visual box size=2.0 1.73 0.76
- added link camera_link; visual box size=0.04 0.03 0.03
- added link front_left_steer_link
- added link front_left_wheel_link; visual cylinder length=0.2 radius=0.315
- added link front_right_steer_link
- added link front_right_wheel_link; visual cylinder length=0.2 radius=0.315
- added link gps_link; visual cylinder length=0.015 radius=0.025
- added link imu_link; visual box size=0.0574 0.0428 0.0235
- added link lidar_link; visual cylinder length=0.0717 radius=0.0517
- added link radar_link; visual box size=0.032 0.09 0.07
- added link rear_left_wheel_link; visual cylinder length=0.2 radius=0.315
- added link rear_right_wheel_link; visual cylinder length=0.2 radius=0.315
Joints:
- added joint body_joint: type fixed, parent base_link, child body_link
- added joint camera_joint: type fixed, parent base_link, child camera_link, origin xyz=1.55 0 1.05 rpy=0 0 0
- added joint front_left_steer_joint: type revolute, parent base_link, child front_left_steer_link, origin xyz=2.648 0.756 -0.085, axis 0 0 1, limit lower=-0.6 upper=0.6 effort=100 velocity=10
- added joint front_left_wheel_joint: type continuous, parent front_left_steer_link, child front_left_wheel_link, axis 0 1 0
- added joint front_right_steer_joint: type revolute, parent base_link, child front_right_steer_link, origin xyz=2.648 -0.756 -0.085, axis 0 0 1, limit lower=-0.6 upper=0.6 effort=100 velocity=10
- added joint front_right_wheel_joint: type continuous, parent front_right_steer_link, child front_right_wheel_link, axis 0 1 0
- added joint gps_joint: type fixed, parent base_link, child gps_link, origin xyz=0.3 0 1.4 rpy=0 0 0
- added joint imu_joint: type fixed, parent base_link, child imu_link, origin xyz=-0.3 0 0.5 rpy=0 0 0
- added joint lidar_joint: type fixed, parent base_link, child lidar_link, origin xyz=0.7 0 1.57 rpy=0 0 0
- added joint radar_joint: type fixed, parent base_link, child radar_link, origin xyz=3.53 -0.06 0.35 rpy=0 0 0
- added joint rear_left_wheel_joint: type continuous, parent base_link, child rear_left_wheel_link, origin xyz=0 0.756 -0.085, axis 0 1 0
- added joint rear_right_wheel_joint: type continuous, parent base_link, child rear_right_wheel_link, origin xyz=0 -0.756 -0.085, axis 0 1 0
